File: pixel-stick.sch (KiCad schematic (older format))
At the start: 21 parts, among them J1 FTDI, J2 WS28**, SW1 RESET, SW2 PROG, U1 AZ1117-3.3, U2 ESP-01v090, U3 SN74LVC1T45DBV, U4 RT9361A

Commit message: add power led
Parts:
- added D2: LED, LED_SMD:LED_1206_3216Metric, symbol Device:LED
- added R4: 120, Resistor_SMD:R_0805_2012Metric, symbol Device:R
Connections:
- wire segments 77 -> 80
Other:
- moved on the sheet: C2, C3, U1
Changed lines of the file:
@@
 EESchema Schematic File Version 4
-LIBS:PixelStickPTH-cache
 EELAYER 29 0
 EELAYER END
@@
 L Regulator_Linear:AZ1117-3.3 U1
 U 1 1 5DE96EF7
-P 2550 1050
-F 0 "U1" H 2550 1292 50  0000 C CNN
-F 1 "AZ1117-3.3" H 2550 1201 50  0000 C CNN
-F 2 "Package_TO_SOT_SMD:SOT-223-3_TabPin2" H 2550 1300 50  0001 C CIN
-F 3 "https://www.diodes.com/assets/Datasheets/AZ1117.pdf" H 2550 1050 50  0001 C CNN
-	1    2550 1050
+P 2200 1050
+F 0 "U1" H 2200 1292 50  0000 C CNN
+F 1 "AZ1117-3.3" H 2200 1201 50  0000 C CNN
+F 2 "Package_TO_SOT_SMD:SOT-223-3_TabPin2" H 2200 1300 50  0001 C CIN
+F 3 "https://www.diodes.com/assets/Datasheets/AZ1117.pdf" H 2200 1050 50  0001 C CNN
+	1    2200 1050
 	1    0    0    -1
 $EndComp
@@
 L power:+VDC #PWR0101
 U 1 1 5DE97D67
-P 1400 1050
-F 0 "#PWR0101" H 1400 950 50  0001 C CNN
-F 1 "+VDC" V 1400 1279 50  0000 L CNN
-F 2 "" H 1400 1050 50  0001 C CNN
-F 3 "" H 1400 1050 50  0001 C CNN
-	1    1400 1050
+P 1050 1050
+F 0 "#PWR0101" H 1050 950 50  0001 C CNN
+F 1 "+VDC" V 1050 1279 50  0000 L CNN
+F 2 "" H 1050 1050 50  0001 C CNN
+F 3 "" H 1050 1050 50  0001 C CNN
+	1    1050 1050
 	0    -1   -1   0
 $EndComp
@@
 L Device:C C2
 U 1 1 5DE99CA9
-P 1800 1350
-F 0 "C2" H 1915 1396 50  0000 L CNN
-F 1 "1µF" H 1915 1305 50  0000 L CNN
-F 2 "Capacitor_SMD:C_0805_2012Metric" H 1838 1200 50  0001 C CNN
-F 3 "~" H 1800 1350 50  0001 C CNN
-	1    1800 1350
+P 1450 1350
+F 0 "C2" H 1565 1396 50  0000 L CNN
+F 1 "1µF" H 1565 1305 50  0000 L CNN
+F 2 "Capacitor_SMD:C_0805_2012Metric" H 1488 1200 50  0001 C CNN
+F 3 "~" H 1450 1350 50  0001 C CNN
+	1    1450 1350
 	1    0    0    -1
 $EndComp
@@
 L Device:C C3
 U 1 1 5DE9A199
-P 3300 1350
-F 0 "C3" H 3415 1396 50  0000 L CNN
-F 1 "10µF" H 3415 1305 50  0000 L CNN
-F 2 "Capacitor_SMD:C_0805_2012Metric" H 3338 1200 50  0001 C CNN
-F 3 "~" H 3300 1350 50  0001 C CNN
-	1    3300 1350
+P 2950 1350
+F 0 "C3" H 3065 1396 50  0000 L CNN
+F 1 "10µF" H 3065 1305 50  0000 L CNN
+F 2 "Capacitor_SMD:C_0805_2012Metric" H 2988 1200 50  0001 C CNN
+F 3 "~" H 2950 1350 50  0001 C CNN
+	1    2950 1350
 	1    0    0    -1
 $EndComp
@@
 L power:GND #PWR0102
 U 1 1 5DE9A40C
-P 2550 1950
-F 0 "#PWR0102" H 2550 1700 50  0001 C CNN
-F 1 "GND" H 2555 1777 50  0000 C CNN
-F 2 "" H 2550 1950 50  0001 C CNN
-F 3 "" H 2550 1950 50  0001 C CNN
-	1    2550 1950
-	1    0    0    -1
-$EndComp
-Wire Wire Line
-	3800 1050 3300 1050
-Wire Wire Line
-	1800 1200 1800 1050
-Wire Wire Line
-	1400 1050 1800 1050
-Connection ~ 1800 1050
-Wire Wire Line
-	1800 1050 2250 1050
-Wire Wire Line
-	1800 1500 1800 1700
-Wire Wire Line
-	1800 1700 2550 1700
-Connection ~ 2550 1700
-Wire Wire Line
-	2550 1700 2550 1350
-Wire Wire Line
-	2550 1700 3300 1700
-Wire Wire Line
-	3300 1700 3300 1500
-Wire Wire Line
-	3300 1200 3300 1050
-Connection ~ 3300 1050
-Wire Wire Line
-	3300 1050 2850 1050
+P 2200 1950
+F 0 "#PWR0102" H 2200 1700 50  0001 C CNN
+F 1 "GND" H 2205 1777 50  0000 C CNN
+F 2 "" H 2200 1950 50  0001 C CNN
+F 3 "" H 2200 1950 50  0001 C CNN
+	1    2200 1950
+	1    0    0    -1
+$EndComp
+Wire Wire Line
+	3450 1050 2950 1050
+Wire Wire Line
+	1450 1200 1450 1050
+Wire Wire Line
+	1050 1050 1450 1050
+Connection ~ 1450 1050
+Wire Wire Line
+	1450 1050 1900 1050
+Wire Wire Line
+	1450 1500 1450 1700
+Wire Wire Line
+	1450 1700 2200 1700
+Connection ~ 2200 1700
+Wire Wire Line
+	2200 1700 2200 1350
+Wire Wire Line
+	2200 1700 2950 1700
+Wire Wire Line
+	2950 1700 2950 1500
+Wire Wire Line
+	2950 1200 2950 1050
+Connection ~ 2950 1050
+Wire Wire Line
+	2950 1050 2500 1050
 $Comp
 L power:+3.3V #PWR0103
 U 1 1 5DE9E6A5
-P 3800 1050
-F 0 "#PWR0103" H 3800 900 50  0001 C CNN
-F 1 "+3.3V" V 3815 1178 50  0000 L CNN
-F 2 "" H 3800 1050 50  0001 C CNN
-F 3 "" H 3800 1050 50  0001 C CNN
-	1    3800 1050
+P 3450 1050
+F 0 "#PWR0103" H 3450 900 50  0001 C CNN
+F 1 "+3.3V" V 3465 1178 50  0000 L CNN
+F 2 "" H 3450 1050 50  0001 C CNN
+F 3 "" H 3450 1050 50  0001 C CNN
+	1    3450 1050
 	0    1    1    0
 $EndComp
@@
 	9100 1400 9300 1400
 Wire Wire Line
-	2550 1950 2550 1700
+	2200 1950 2200 1700
 $Comp
 L power:GND #PWR0113
@@
 Wire Wire Line
 	6600 3600 7150 3600
+$Comp
+L power:+3.3V #PWR0123
+U 1 1 5DED69A9
+P 4100 1000
+F 0 "#PWR0123" H 4100 850 50  0001 C CNN
+F 1 "+3.3V" V 4115 1128 50  0000 L CNN
+F 2 "" H 4100 1000 50  0001 C CNN
+F 3 "" H 4100 1000 50  0001 C CNN
+	1    4100 1000
+	1    0    0    -1
+$EndComp
+$Comp
+L power:GND #PWR0124
+U 1 1 5DED69AF
+P 4100 2050
+F 0 "#PWR0124" H 4100 1800 50  0001 C CNN
+F 1 "GND" H 4105 1877 50  0000 C CNN
+F 2 "" H 4100 2050 50  0001 C CNN
+F 3 "" H 4100 2050 50  0001 C CNN
+	1    4100 2050
+	1    0    0    -1
+$EndComp
+$Comp
+L Device:R R4
+U 1 1 5DEDDC6F
+P 4100 1300
+F 0 "R4" V 3893 1300 50  0000 C CNN
+F 1 "120" V 3984 1300 50  0000 C CNN
+F 2 "Resistor_SMD:R_0805_2012Metric" V 4030 1300 50  0001 C CNN
+F 3 "~" H 4100 1300 50  0001 C CNN
+	1    4100 1300
+	-1   0    0    1
+$EndComp
+Wire Wire Line
+	4100 1000 4100 1150
+Wire Wire Line
+	4100 1450 4100 1600
+$Comp
+L Device:LED D2
+U 1 1 5DEF1859
+P 4100 1750
+F 0 "D2" V 4139 1633 50  0000 R CNN
+F 1 "LED" V 4048 1633 50  0000 R CNN
+F 2 "LED_SMD:LED_1206_3216Metric" H 4100 1750 50  0001 C CNN
+F 3 "~" H 4100 1750 50  0001 C CNN
+	1    4100 1750
+	0    -1   -1   0
+$EndComp
+Wire Wire Line
+	4100 1900 4100 2050
 $EndSCHEMATC

Commit message: fix drc errors
Changed lines of the file:
@@
 VIN
 Text Label 10250 1150 0    50   ~ 0
+CLOCK
+Text Label 10250 1250 0    50   ~ 0
 DATA
-Text Label 10250 1250 0    50   ~ 0
-CLOCK
 Text Label 10250 1350 0    50   ~ 0
 GND

Commit message: remove programming features
Parts:
- removed C4: 10µF, Capacitor_SMD:C_0805_2012Metric, symbol Device:C
- removed D1: 1N5819, Diode_SMD:D_SOD-123, symbol Diode:1N5819
- removed J1: FTDI, Connector_PinHeader_1.00mm:PinHeader_1x06_P1.00mm_Vertical, symbol Connector_Generic:Conn_01x06
- removed R2: 10k, Resistor_SMD:R_0805_2012Metric, symbol Device:R
- removed SW1: RESET, Button_Switch_SMD:SW_SPST_TL3305A, symbol Switch:SW_SPST
- removed SW2: PROG, Button_Switch_SMD:SW_SPST_TL3305A, symbol Switch:SW_SPST
Connections:
- net labels removed: RXD_5V, VDC
- wire segments 80 -> 63
Other:
- note removed: "BUTTONS"
- note removed: "FTDI"
- moved on the sheet: C1, R1

Commit message: cleanup silkscreen layer
Parts:
- removed R1: 10k, Resistor_SMD:R_0805_2012Metric, symbol Device:R
Connections:
- net labels removed: ~RST
- wire segments 63 -> 62
Other:
- moved on the sheet: C1, U2
Changed lines of the file:
@@
 L ESP8266:ESP-01v090 U2
 U 1 1 5DE9E498
-P 2850 3450
-F 0 "U2" H 2850 4000 50  0000 C CNN
-F 1 "ESP-01v090" H 2850 3900 50  0000 C CNN
-F 2 "ESP8266:ESP-01" H 2850 3450 50  0001 C CNN
-F 3 "http://l0l.org.uk/2014/12/esp8266-modules-hardware-guide-gotta-catch-em-all/" H 2850 3450 50  0001 C CNN
-	1    2850 3450
+P 2700 3450
+F 0 "U2" H 2700 4000 50  0000 C CNN
+F 1 "ESP-01v090" H 2700 3900 50  0000 C CNN
+F 2 "ESP8266:ESP-01" H 2700 3450 50  0001 C CNN
+F 3 "http://l0l.org.uk/2014/12/esp8266-modules-hardware-guide-gotta-catch-em-all/" H 2700 3450 50  0001 C CNN
+	1    2700 3450
 	1    0    0    -1
 $EndComp
@@
 L Device:C C1
 U 1 1 5DE9F007
-P 800 3800
-F 0 "C1" H 915 3846 50  0000 L CNN
-F 1 "10µF" H 915 3755 50  0000 L CNN
-F 2 "Capacitor_SMD:C_0805_2012Metric" H 838 3650 50  0001 C CNN
-F 3 "~" H 800 3800 50  0001 C CNN
-	1    800  3800
+P 1000 3700
+F 0 "C1" H 1115 3746 50  0000 L CNN
+F 1 "10µF" H 1115 3655 50  0000 L CNN
+F 2 "Capacitor_SMD:C_0805_2012Metric" H 1038 3550 50  0001 C CNN
+F 3 "~" H 1000 3700 50  0001 C CNN
+	1    1000 3700
 	1    0    0    -1
 $EndComp
@@
 L power:+3.3V #PWR0104
 U 1 1 5DE9F73D
-P 800 3300
-F 0 "#PWR0104" H 800 3150 50  0001 C CNN
-F 1 "+3.3V" V 815 3428 50  0000 L CNN
-F 2 "" H 800 3300 50  0001 C CNN
-F 3 "" H 800 3300 50  0001 C CNN
-	1    800  3300
+P 1000 3200
+F 0 "#PWR0104" H 1000 3050 50  0001 C CNN
+F 1 "+3.3V" V 1015 3328 50  0000 L CNN
+F 2 "" H 1000 3200 50  0001 C CNN
+F 3 "" H 1000 3200 50  0001 C CNN
+	1    1000 3200
 	1    0    0    -1
 $EndComp
@@
 L power:GND #PWR0105
 U 1 1 5DEA0257
-P 800 4350
-F 0 "#PWR0105" H 800 4100 50  0001 C CNN
-F 1 "GND" H 805 4177 50  0000 C CNN
-F 2 "" H 800 4350 50  0001 C CNN
-F 3 "" H 800 4350 50  0001 C CNN
-	1    800  4350
+P 1000 4250
+F 0 "#PWR0105" H 1000 4000 50  0001 C CNN
+F 1 "GND" H 1005 4077 50  0000 C CNN
+F 2 "" H 1000 4250 50  0001 C CNN
+F 3 "" H 1000 4250 50  0001 C CNN
+	1    1000 4250
 	1    0    0    -1
 $EndComp
@@
 L power:GND #PWR0106
 U 1 1 5DEA2B31
-P 2850 4350
-F 0 "#PWR0106" H 2850 4100 50  0001 C CNN
-F 1 "GND" H 2855 4177 50  0000 C CNN
-F 2 "" H 2850 4350 50  0001 C CNN
-F 3 "" H 2850 4350 50  0001 C CNN
-	1    2850 4350
-	1    0    0    -1
-$EndComp
-Wire Wire Line
-	2850 4350 2850 4200
-Wire Wire Line
-	3600 3400 3950 3400
-Wire Wire Line
-	3600 3550 3950 3550
-Wire Wire Line
-	3600 3800 3950 3800
-Wire Wire Line
-	3600 3950 3950 3950
-Wire Wire Line
-	2100 3400 2000 3400
-Wire Wire Line
-	2100 3550 2000 3550
-Wire Wire Line
-	2100 3700 1750 3700
-Text Label 1950 3700 2    50   ~ 0
-~RST
-Text Label 3700 3400 0    50   ~ 0
+P 2700 4350
+F 0 "#PWR0106" H 2700 4100 50  0001 C CNN
+F 1 "GND" H 2705 4177 50  0000 C CNN
+F 2 "" H 2700 4350 50  0001 C CNN
+F 3 "" H 2700 4350 50  0001 C CNN
+	1    2700 4350
+	1    0    0    -1
+$EndComp
+Wire Wire Line
+	2700 4350 2700 4200
+Wire Wire Line
+	3450 3400 3800 3400
+Wire Wire Line
+	3450 3550 3800 3550
+Wire Wire Line
+	3450 3800 3800 3800
+Wire Wire Line
+	3450 3950 3800 3950
+Wire Wire Line
+	1950 3400 1850 3400
+Wire Wire Line
+	1950 3550 1850 3550
+Text Label 3550 3400 0    50   ~ 0
 GPIO2
-Text Label 3700 3550 0    50   ~ 0
+Text Label 3550 3550 0    50   ~ 0
 GPIO0
-Text Label 3700 3800 0    50   ~ 0
+Text Label 3550 3800 0    50   ~ 0
 TXD
-Text Label 3700 3950 0    50   ~ 0
+Text Label 3550 3950 0    50   ~ 0
 RXD
 $Comp
 L power:+3.3V #PWR0107
 U 1 1 5DEA7FFE
-P 1950 3400
-F 0 "#PWR0107" H 1950 3250 50  0001 C CNN
-F 1 "+3.3V" V 1965 3528 50  0000 L CNN
-F 2 "" H 1950 3400 50  0001 C CNN
-F 3 "" H 1950 3400 50  0001 C CNN
-	1    1950 3400
+P 1800 3400
+F 0 "#PWR0107" H 1800 3250 50  0001 C CNN
+F 1 "+3.3V" V 1815 3528 50  0000 L CNN
+F 2 "" H 1800 3400 50  0001 C CNN
+F 3 "" H 1800 3400 50  0001 C CNN
+	1    1800 3400
 	0    -1   -1   0
 $EndComp
 Wire Wire Line
-	800  3300 800  3650
-Wire Wire Line
-	800  3950 800  4350
+	1000 3200 1000 3550
+Wire Wire Line
+	1000 3850 1000 4250
 Wire Notes Line
 	500  5050 4550 5050
 Wire Wire Line
-	2000 3400 2000 3550
-Connection ~ 2000 3400
-Wire Wire Line
-	2000 3400 1950 3400
+	1850 3400 1850 3550
+Connection ~ 1850 3400
+Wire Wire Line
+	1850 3400 1800 3400
 $Comp
 L Regulator_Linear:AP3602A U4
@@
 Text Notes 8700 2500 0    157  ~ 0
 Input / Protection
-$Comp
-L power:+3.3V #PWR0114
-U 1 1 5DF05847
-P 1300 3300
-F 0 "#PWR0114" H 1300 3150 50  0001 C CNN
-F 1 "+3.3V" V 1315 3428 50  0000 L CNN
-F 2 "" H 1300 3300 50  0001 C CNN
-F 3 "" H 1300 3300 50  0001 C CNN
-	1    1300 3300
-	1    0    0    -1
-$EndComp
-$Comp
-L Device:R R1
-U 1 1 5DF0756F
-P 1300 3750
-F 0 "R1" V 1093 3750 50  0000 C CNN
-F 1 "10k" V 1184 3750 50  0000 C CNN
-F 2 "Resistor_SMD:R_0805_2012Metric" V 1230 3750 50  0001 C CNN
-F 3 "~" H 1300 3750 50  0001 C CNN
-	1    1300 3750
-	-1   0    0    1
-$EndComp
-Wire Wire Line
-	1300 3300 1300 3600
-Wire Wire Line
-	1300 3900 1300 4450
-Text Label 1300 4200 3    50   ~ 0
-~RST
 Wire Notes Line
 	4550 500  4550 5050
@@
 Wire Wire Line
 	5300 1000 5950 1000
+Wire Wire Line
+	1950 3700 1850 3700
+Wire Wire Line
+	1850 3700 1850 3550
+Connection ~ 1850 3550
 $EndSCHEMATC

Commit message: replace logic chip with simple buffer
Parts:
- removed R3: 10k, Resistor_SMD:R_0805_2012Metric, symbol Device:R
- removed U3: SN74LVC1T45DBV, Package_TO_SOT_SMD:SOT-23-6, symbol Logic_LevelTranslator:SN74LVC1T45DBV
- added U4: 74AHC1G125, Package_TO_SOT_SMD:SOT-23-5, symbol 74xGxx:74AHC1G125
- renumbered C2 to C1, C3 to C2, C6 to C3, C5 to C4, C7 to C5, C1 to C6, D2 to D1, J2 to J1, R4 to R1, U4 to U1, U1 to U2, U2 to U3
Connections:
- wire segments 62 -> 60

Commit message: increase passives to 1206 footprint
Parts:
- U2: renamed from U1; value RT9361A -> RT9361AGE
- U3: renamed from U4; value 74AHC1G125 -> MC74VHC1GT125
- renumbered C5 to C1, C1 to C2, C2 to C3, C3 to C5, U3 to ESP-01, U2 to U1
Connections:
- net labels removed: +VDC
- wire segments 60 -> 59
Other:
- note added: "Power Management"
- note removed: "3.3V Power Supply"
- note removed: "5V Power Supply"
- note removed: "Input / Protection"
- moved on the sheet: C1, C2, C3, C4, C5, C6, ESP-01, R1, U1

Commit message: cleanup
Parts:
- removed D1: LED, LED_SMD:LED_1206_3216Metric, symbol Device:LED
- removed J1: WS28**, Connector_PinHeader_1.00mm:PinHeader_1x04_P1.00mm_Vertical, symbol Connector_Generic:Conn_01x04
- removed NT1: Net-Tie_2, NetTie:NetTie-2_SMD_Pad0.5mm, symbol Device:Net-Tie_2
- removed R1: 120, Resistor_SMD:R_0805_2012Metric, symbol Device:R
- added J1: WS2811, Connector_Wire:SolderWirePad_1x03_P3.81mm_Drill1.2mm, symbol Connector_Generic:Conn_01x03
- C1: footprint Capacitor_SMD:CP_Elec_8x5.4 -> Capacitor_SMD:CP_Elec_6.3x7.7
- C2, C3, C4, C5, C6: footprint Capacitor_SMD:C_0805_2012Metric -> Capacitor_SMD:C_1206_3216Metric_Pad1.42x1.75mm_HandSolder
- F1: footprint Resistor_SMD:R_1206_3216Metric -> Resistor_SMD:R_1206_3216Metric_Pad1.42x1.75mm_HandSolder
- U2: footprint Package_TO_SOT_SMD:SOT-23-6 -> Package_TO_SOT_SMD:SOT-23-6_Handsoldering
- U3: footprint Package_TO_SOT_SMD:SOT-23-5 -> Package_TO_SOT_SMD:SOT-23-5_HandSoldering
Connections:
- net labels removed: CLOCK
- wire segments 59 -> 53
Other:
- note added: "VIN between 4.5 and 15VDC. \nData is 5V CMOS logic."
- note removed: "VIN between 4.5 and 15VDC. \nData and Clock are 5V CMOS\nlogic compatible."
Changed lines of the file:
@@
 F 0 "C2" H 4915 1996 50  0000 L CNN
 F 1 "1µF" H 4915 1905 50  0000 L CNN
-F 2 "Capacitor_SMD:C_0805_2012Metric" H 4838 1800 50  0001 C CNN
+F 2 "Capacitor_SMD:C_1206_3216Metric_Pad1.42x1.75mm_HandSolder" H 4838 1800 50  0001 C CNN
 F 3 "~" H 4800 1950 50  0001 C CNN
 	1    4800 1950
@@
 F 0 "C3" H 6415 1996 50  0000 L CNN
 F 1 "10µF" H 6415 1905 50  0000 L CNN
-F 2 "Capacitor_SMD:C_0805_2012Metric" H 6338 1800 50  0001 C CNN
+F 2 "Capacitor_SMD:C_1206_3216Metric_Pad1.42x1.75mm_HandSolder" H 6338 1800 50  0001 C CNN
 F 3 "~" H 6300 1950 50  0001 C CNN
 	1    6300 1950
@@
 F 0 "U2" H 7250 1450 50  0000 C CNN
 F 1 "RT9361AGE" H 7250 1350 50  0000 C CNN
-F 2 "Package_TO_SOT_SMD:SOT-23-6" H 7250 1383 50  0001 C CNN
+F 2 "Package_TO_SOT_SMD:SOT-23-6_Handsoldering" H 7250 1383 50  0001 C CNN
 F 3 "https://www.richtek.com/assets/product_file/RT9361A=RT9361B/DS9361AB-14.pdf" H 7250 1450 50  0001 C CNN
 	1    7250 1450
@@
 	8350 2300 7900 2300
 Connection ~ 8350 2300
-Wire Wire Line
-	1250 1250 1600 1250
-Wire Wire Line
-	1250 1350 1600 1350
-Wire Wire Line
-	1250 1450 1600 1450
-Wire Wire Line
-	1250 1550 1600 1550
-Text Label 1300 1250 0    50   ~ 0
-VIN
-Text Label 1300 1350 0    50   ~ 0
-CLOCK
-Text Label 1300 1450 0    50   ~ 0
-DATA
-Text Label 1300 1550 0    50   ~ 0
-GND
 $Comp
 L Device:Polyfuse F1
@@
 F 0 "F1" V 3800 1600 50  0000 L CNN
 F 1 "Polyfuse" V 3550 1500 50  0000 L CNN
-F 2 "Resistor_SMD:R_1206_3216Metric" H 3750 1450 50  0001 L CNN
+F 2 "Resistor_SMD:R_1206_3216Metric_Pad1.42x1.75mm_HandSolder" H 3750 1450 50  0001 L CNN
 F 3 "~" H 3700 1650 50  0001 C CNN
 	1    3700 1650
@@
 F 0 "C5" H 8465 2046 50  0000 L CNN
 F 1 "10µF" H 8465 1955 50  0000 L CNN
-F 2 "Capacitor_SMD:C_0805_2012Metric" H 8388 1850 50  0001 C CNN
+F 2 "Capacitor_SMD:C_1206_3216Metric_Pad1.42x1.75mm_HandSolder" H 8388 1850 50  0001 C CNN
 F 3 "~" H 8350 2000 50  0001 C CNN
 	1    8350 2000
@@
 F 0 "C1" H 4265 2046 50  0000 L CNN
 F 1 "100µF" H 4265 1955 50  0000 L CNN
-F 2 "Capacitor_SMD:CP_Elec_8x5.4" H 4150 2000 50  0001 C CNN
+F 2 "Capacitor_SMD:CP_Elec_6.3x7.7" H 4150 2000 50  0001 C CNN
 F 3 "~" H 4150 2000 50  0001 C CNN
 	1    4150 2000
@@
 Wire Wire Line
 	4150 2150 4150 2500
-Text Notes 1000 1950 0    50   ~ 0
-VIN between 4.5 and 15VDC. \nData and Clock are 5V CMOS\nlogic compatible.
-$Comp
-L Connector_Generic:Conn_01x04 J1
-U 1 1 5DF54B71
-P 1800 1350
-F 0 "J1" H 1880 1342 50  0000 L CNN
-F 1 "WS28**" H 1880 1251 50  0000 L CNN
-F 2 "Connector_PinHeader_1.00mm:PinHeader_1x04_P1.00mm_Vertical" H 1800 1350 50  0001 C CNN
-F 3 "~" H 1800 1350 50  0001 C CNN
-	1    1800 1350
-	1    0    0    -1
-$EndComp
+Text Notes 1200 2200 0    50   ~ 0
+VIN between 4.5 and 15VDC. \nData is 5V CMOS logic.
 Wire Wire Line
 	4150 1650 4150 1850
-$Comp
-L power:+3.3V #PWR03
-U 1 1 5DED69A9
-P 10100 1350
-F 0 "#PWR03" H 10100 1200 50  0001 C CNN
-F 1 "+3.3V" V 10115 1478 50  0000 L CNN
-F 2 "" H 10100 1350 50  0001 C CNN
-F 3 "" H 10100 1350 50  0001 C CNN
-	1    10100 1350
-	1    0    0    -1
-$EndComp
-$Comp
-L power:GND #PWR06
-U 1 1 5DED69AF
-P 10100 2500
-F 0 "#PWR06" H 10100 2250 50  0001 C CNN
-F 1 "GND" H 10105 2327 50  0000 C CNN
-F 2 "" H 10100 2500 50  0001 C CNN
-F 3 "" H 10100 2500 50  0001 C CNN
-	1    10100 2500
-	1    0    0    -1
-$EndComp
-$Comp
-L Device:R R1
-U 1 1 5DEDDC6F
-P 10100 1700
-F 0 "R1" V 9893 1700 50  0000 C CNN
-F 1 "120" V 9984 1700 50  0000 C CNN
-F 2 "Resistor_SMD:R_0805_2012Metric" V 10030 1700 50  0001 C CNN
-F 3 "~" H 10100 1700 50  0001 C CNN
-	1    10100 1700
-	-1   0    0    1
-$EndComp
-Wire Wire Line
-	10100 1350 10100 1550
-Wire Wire Line
-	10100 1850 10100 2000
-$Comp
-L Device:LED D1
-U 1 1 5DEF1859
-P 10100 2150
-F 0 "D1" V 10139 2033 50  0000 R CNN
-F 1 "LED" V 10048 2033 50  0000 R CNN
-F 2 "LED_SMD:LED_1206_3216Metric" H 10100 2150 50  0001 C CNN
-F 3 "~" H 10100 2150 50  0001 C CNN
-	1    10100 2150
-	0    -1   -1   0
-$EndComp
-Wire Wire Line
-	10100 2300 10100 2500
 $Comp
 L power:+3.3V #PWR01
@@
 F 0 "U3" H 7725 4725 50  0000 C CNN
 F 1 "MC74VHC1GT125" H 7725 4634 50  0000 C CNN
-F 2 "Package_TO_SOT_SMD:SOT-23-5" H 7750 4900 50  0001 C CNN
+F 2 "Package_TO_SOT_SMD:SOT-23-5_HandSoldering" H 7750 4900 50  0001 C CNN
 F 3 "https://www.onsemi.com/pub/Collateral/MC74VHC1GT125-D.PDF" H 7750 4900 50  0001 C CNN
 	1    7750 4900
 	1    0    0    -1
-$EndComp
-Text Label 8900 5200 1    50   ~ 0
-CLOCK
-Text Label 8900 4350 3    50   ~ 0
-GPIO0
-Wire Wire Line
-	8900 4700 8900 4350
-Wire Wire Line
-	8900 4900 8900 5200
-$Comp
-L Device:Net-Tie_2 NT1
-U 1 1 5E05448E
-P 8900 4800
-F 0 "NT1" H 8900 4981 50  0001 C CNN
-F 1 "Net-Tie_2" H 8900 4890 50  0001 C CNN
-F 2 "NetTie:NetTie-2_SMD_Pad0.5mm" H 8900 4800 50  0001 C CNN
-F 3 "~" H 8900 4800 50  0001 C CNN
-	1    8900 4800
-	0    1    1    0
 $EndComp
 Text Notes 7100 6050 0    157  ~ 0
@@
 F 0 "C6" H 1465 4896 50  0000 L CNN
 F 1 "10µF" H 1465 4805 50  0000 L CNN
-F 2 "Capacitor_SMD:C_0805_2012Metric" H 1388 4700 50  0001 C CNN
+F 2 "Capacitor_SMD:C_1206_3216Metric_Pad1.42x1.75mm_HandSolder" H 1388 4700 50  0001 C CNN
 F 3 "~" H 1350 4850 50  0001 C CNN
 	1    1350 4850
@@
 F 0 "C4" V 7100 2400 50  0000 C CNN
 F 1 "1µF" V 7400 2400 50  0000 C CNN
-F 2 "Capacitor_SMD:C_0805_2012Metric" H 7288 2250 50  0001 C CNN
+F 2 "Capacitor_SMD:C_1206_3216Metric_Pad1.42x1.75mm_HandSolder" H 7288 2250 50  0001 C CNN
 F 3 "~" H 7250 2400 50  0001 C CNN
 	1    7250 2400
 	0    1    1    0
 $EndComp
+$Comp
+L Connector_Generic:Conn_01x03 J1
+U 1 1 5DFF0485
+P 1900 1700
+F 0 "J1" H 1980 1742 50  0000 L CNN
+F 1 "WS2811" H 1980 1651 50  0000 L CNN
+F 2 "Connector_Wire:SolderWirePad_1x03_P3.81mm_Drill1.2mm" H 1900 1700 50  0001 C CNN
+F 3 "~" H 1900 1700 50  0001 C CNN
+	1    1900 1700
+	1    0    0    -1
+$EndComp
+Wire Wire Line
+	1250 1600 1700 1600
+Text Label 1300 1800 0    50   ~ 0
+GND
+Text Label 1300 1700 0    50   ~ 0
+DATA
+Text Label 1300 1600 0    50   ~ 0
+VIN
+Wire Wire Line
+	1250 1800 1700 1800
+Wire Wire Line
+	1250 1700 1700 1700
 $EndSCHEMATC

Commit message: make custom vin power symbol
Connections:
- wire segments 53 -> 56
Changed lines of the file:
@@
 Wire Wire Line
 	3550 1650 3200 1650
-Text Label 3350 1650 2    50   ~ 0
-VIN
 $Comp
 L power:GND #PWR05
@@
 Wire Wire Line
 	4150 2150 4150 2500
-Text Notes 1200 2200 0    50   ~ 0
+Text Notes 1200 2400 0    50   ~ 0
 VIN between 4.5 and 15VDC. \nData is 5V CMOS logic.
 Wire Wire Line
@@
 	1    0    0    -1
 $EndComp
-Wire Wire Line
-	1250 1600 1700 1600
-Text Label 1300 1800 0    50   ~ 0
-GND
 Text Label 1300 1700 0    50   ~ 0
 DATA
-Text Label 1300 1600 0    50   ~ 0
-VIN
-Wire Wire Line
-	1250 1800 1700 1800
 Wire Wire Line
 	1250 1700 1700 1700
+$Comp
+L power:VIN #PWR?
+U 1 1 5DFA6142
+P 1550 1500
+F 0 "#PWR?" H 1550 1350 50  0001 C CNN
+F 1 "VIN" H 1565 1673 50  0000 C CNN
+F 2 "" H 1550 1500 50  0001 C CNN
+F 3 "" H 1550 1500 50  0001 C CNN
+	1    1550 1500
+	1    0    0    -1
+$EndComp
+$Comp
+L power:GND #PWR?
+U 1 1 5DFA6D40
+P 1550 1900
+F 0 "#PWR?" H 1550 1650 50  0001 C CNN
+F 1 "GND" H 1555 1727 50  0000 C CNN
+F 2 "" H 1550 1900 50  0001 C CNN
+F 3 "" H 1550 1900 50  0001 C CNN
+	1    1550 1900
+	1    0    0    -1
+$EndComp
+Wire Wire Line
+	1550 1500 1550 1600
+Wire Wire Line
+	1550 1600 1700 1600
+Wire Wire Line
+	1550 1900 1550 1800
+Wire Wire Line
+	1550 1800 1700 1800
+$Comp
+L power:VIN #PWR?
+U 1 1 5DFAB074
+P 3200 1500
+F 0 "#PWR?" H 3200 1350 50  0001 C CNN
+F 1 "VIN" H 3215 1673 50  0000 C CNN
+F 2 "" H 3200 1500 50  0001 C CNN
+F 3 "" H 3200 1500 50  0001 C CNN
+	1    3200 1500
+	1    0    0    -1
+$EndComp
+Wire Wire Line
+	3200 1500 3200 1650
 $EndSCHEMATC
